File: hardware/teste_estatico/kicad/teste_estatico.kicad_pcb (KiCad board)
At the start: 2 copper layers, 10 parts

Commit message: adcionado atulização nos arquivos de pcb kicad
Parts:
- moved R3.3k1 65.7 mm to (196.2, 126.2), turned to 180 degrees
- moved SDCARD1 59.8 mm to (81.2, 80.0)
- moved PRESSÃO1 52.8 mm to (191.2, 74.7)
- moved R2.2k1 45.6 mm to (157.5, 126.2)
- moved R220ohn1 37.9 mm to (132.3, 126.8)
- moved D1 37.5 mm to (111.0, 126.8)
- moved tara1 35.2 mm to (171.5, 97.5)
- moved RJ45 33.9 mm to (162.2, 73.5), turned to 90 degrees
- moved NOVOARQUIVO1 32.1 mm to (154.0, 97.5)
Routing:
- net Net-(A1-ADC1_CH7/D35): track 0.00 -> 89.0 mm
- net Net-(A1-ADC1_CH4/D32-Pad22): track 0.00 -> 6.50 mm
- net Net-(A1-ADC1_CH4/D32-Pad21): track 0.00 -> 6.50 mm
Changed lines of the file:
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@@
 	(footprint "PCM_SL_Development_Boards:DOIT_ESP32_DEVKIT_30Pins"
 		(layer "F.Cu")
-		(at 109.566929 76.24)
+		(at 109.5669 76.24)
 		(property "Reference" "A1"
 			(at 13.253071 1.86 0)
@@
 	(footprint "Button_Switch_THT:SW_PUSH_6mm"
 		(layer "F.Cu")
-		(at 143.96 66.99)
+		(at 154 97.5)
 		(descr "Generic 6mm SW tactile push button")
 		(tags "tact sw push 6mm")
@@
 	(footprint "Button_Switch_THT:SW_PUSH_6mm"
 		(layer "F.Cu")
-		(at 143.96 75.54)
+		(at 171.5 97.5)
 		(descr "Generic 6mm SW tactile push button")
 		(tags "tact sw push 6mm")
@@
 	(footprint "Connector_PinSocket_2.54mm:PinSocket_1x06_P2.54mm_Vertical"
 		(layer "F.Cu")
-		(at 139.66 67.29)
+		(at 81.25 80.05)
 		(descr "Through hole straight socket strip, 1x06, 2.54mm pitch, single row (from Kicad 4.0.7), script generated")
 		(tags "Through hole socket strip THT 1x06 2.54mm single row")
@@
 		(pad "2" thru_hole circle
 			(at 0 2.54)
-			(size 1.7 1.7)
+			(size 2.5 2.5)
 			(drill 1)
 			(layers "*.Cu" "*.Mask")
@@
 		(pad "3" thru_hole circle
 			(at 0 5.08)
-			(size 1.7 1.7)
+			(size 2.5 2.5)
 			(drill 1)
 			(layers "*.Cu" "*.Mask")
@@
 		(pad "4" thru_hole circle
 			(at 0 7.62)
-			(size 1.7 1.7)
+			(size 2.5 2.5)
 			(drill 1)
 			(layers "*.Cu" "*.Mask")
@@
 		(pad "5" thru_hole circle
 			(at 0 10.16)
-			(size 1.7 1.7)
+			(size 2.5 2.5)
 			(drill 1)
 			(layers "*.Cu" "*.Mask")
@@
 		(pad "6" thru_hole circle
 			(at 0 12.7)
-			(size 1.7 1.7)
+			(size 2.5 2.5)
 			(drill 1)
 			(layers "*.Cu" "*.Mask")
@@
 	(footprint "LED_THT:LED_D5.0mm_FlatTop"
 		(layer "F.Cu")
-		(at 144.46 110)
+		(at 110.96 126.75)
 		(descr "LED, Round, Flat Top, diameter 5.0mm, 2 pins, https://www.kingbright.com/attachments/file/psearch/000/00/watermark00/L-483GDT(Ver.12B).pdf, generated by kicad-footprint-generator")
 		(tags "LED")
@@
 	(footprint "Resistor_THT:R_Axial_DIN0309_L9.0mm_D3.2mm_P12.70mm_Horizontal"
 		(layer "F.Cu")
-		(at 138.91 89.39)
+		(at 132.3 126.75)
 		(descr "Resistor, Axial_DIN0309 series, Axial, Horizontal, pin pitch=12.7mm, 0.5W = 1/2W, length*diameter=9*3.2mm^2, http://cdn-reichelt.de/documents/datenblatt/B400/1_4W%23YAG.pdf")
 		(tags "Resistor Axial_DIN0309 series Axial Horizontal pin pitch 12.7mm 0.5W = 1/2W length 9mm diameter 3.2mm")
@@
 	(footprint "Connector_PinSocket_2.54mm:PinSocket_1x04_P2.54mm_Vertical"
 		(layer "F.Cu")
-		(at 139.66 98.84)
+		(at 162.25 73.5 90)
 		(descr "Through hole straight socket strip, 1x04, 2.54mm pitch, single row (from Kicad 4.0.7), script generated")
 		(tags "Through hole socket strip THT 1x04 2.54mm single row")
 		(property "Reference" "RJ45"
-			(at 0 -2.77 0)
+			(at 0 -2.77 90)
 			(layer "F.SilkS")
 			(effects
@@
 		)
 		(property "Value" "conexão do rj45"
-			(at 0 10.39 0)
+			(at 0 10.39 90)
 			(layer "F.Fab")
 			(effects
@@
 		)
 		(property "Datasheet" ""
-			(at 0 0 0)
+			(at 0 0 90)
 			(layer "F.Fab")
 			(hide yes)
@@
 		)
 		(property "Description" "Pin Header female with pin space 2.54mm. Pin Count -4"
-			(at 0 0 0)
+			(at 0 0 90)
 			(layer "F.Fab")
 			(hide yes)
@@
 		(attr through_hole)
 		(fp_line
-			(start -1.33 1.27)
-			(end -1.33 8.95)
+			(start 1.33 -1.33)
+			(end 1.33 0)
 			(stroke
 				(width 0.12)
@@
 		)
 		(fp_line
-			(start -1.33 1.27)
-			(end 1.33 1.27)
+			(start 0 -1.33)
+			(end 1.33 -1.33)
 			(stroke
 				(width 0.12)
@@
 		)
 		(fp_line
-			(start -1.33 8.95)
+			(start 1.33 1.27)
 			(end 1.33 8.95)
 			(stroke
@@
 		)
 		(fp_line
-			(start 0 -1.33)
-			(end 1.33 -1.33)
+			(start -1.33 1.27)
+			(end 1.33 1.27)
 			(stroke
 				(width 0.12)
@@
 		)
 		(fp_line
-			(start 1.33 -1.33)
-			(end 1.33 0)
+			(start -1.33 1.27)
+			(end -1.33 8.95)
 			(stroke
 				(width 0.12)
@@
 		)
 		(fp_line
-			(start 1.33 1.27)
+			(start -1.33 8.95)
 			(end 1.33 8.95)
 			(stroke
@@
 		)
 		(fp_line
-			(start -1.8 -1.8)
-			(end 1.75 -1.8)
+			(start 1.75 -1.8)
+			(end 1.75 9.4)
 			(stroke
 				(width 0.05)
@@
 		)
 		(fp_line
-			(start -1.8 9.4)
-			(end -1.8 -1.8)
+			(start -1.8 -1.8)
+			(end 1.75 -1.8)
 			(stroke
 				(width 0.05)
@@
 		)
 		(fp_line
-			(start 1.75 -1.8)
-			(end 1.75 9.4)
+			(start 1.75 9.4)
+			(end -1.8 9.4)
 			(stroke
 				(width 0.05)
@@
 		)
 		(fp_line
-			(start 1.75 9.4)
-			(end -1.8 9.4)
+			(start -1.8 9.4)
+			(end -1.8 -1.8)
 			(stroke
 				(width 0.05)
@@
 		)
 		(fp_line
-			(start -1.27 -1.27)
-			(end 0.635 -1.27)
+			(start 0.635 -1.27)
+			(end 1.27 -0.635)
 			(stroke
 				(width 0.1)
@@
 		)
 		(fp_line
-			(start -1.27 8.89)
-			(end -1.27 -1.27)
+			(start -1.27 -1.27)
+			(end 0.635 -1.27)
 			(stroke
 				(width 0.1)
@@
 		)
 		(fp_line
-			(start 0.635 -1.27)
-			(end 1.27 -0.635)
+			(start 1.27 -0.635)
+			(end 1.27 8.89)
 			(stroke
 				(width 0.1)
@@
 		)
 		(fp_line
-			(start 1.27 -0.635)
-			(end 1.27 8.89)
+			(start 1.27 8.89)
+			(end -1.27 8.89)
 			(stroke
 				(width 0.1)
@@
 		)
 		(fp_line
-			(start 1.27 8.89)
-			(end -1.27 8.89)
+			(start -1.27 8.89)
+			(end -1.27 -1.27)
 			(stroke
 				(width 0.1)
@@
 		)
 		(fp_text user "${REFERENCE}"
-			(at 0 3.81 90)
+			(at 0 3.81 0)
 			(layer "F.Fab")
 			(effects
@@
 		)
 		(pad "1" thru_hole rect
-			(at 0 0)
+			(at 0 0 90)
 			(size 1.7 1.7)
 			(drill 1)
@@
 		)
 		(pad "2" thru_hole circle
-			(at 0 2.54)
+			(at 0 2.54 90)
 			(size 1.7 1.7)
 			(drill 1)
@@
 		)
 		(pad "3" thru_hole circle
-			(at 0 5.08)
+			(at 0 5.08 90)
 			(size 1.7 1.7)
 			(drill 1)
@@
 		)
 		(pad "4" thru_hole circle
-			(at 0 7.62)
+			(at 0 7.62 90)
 			(size 1.7 1.7)
 			(drill 1)
@@
 	(footprint "Resistor_THT:R_Axial_DIN0309_L9.0mm_D3.2mm_P12.70mm_Horizontal"
 		(layer "F.Cu")
-		(at 138.91 84.64)
+		(at 157.5 126.25)
 		(descr "Resistor, Axial_DIN0309 series, Axial, Horizontal, pin pitch=12.7mm, 0.5W = 1/2W, length*diameter=9*3.2mm^2, http://cdn-reichelt.de/documents/datenblatt/B400/1_4W%23YAG.pdf")
 		(tags "Resistor Axial_DIN0309 series Axial Horizontal pin pitch 12.7mm 0.5W = 1/2W length 9mm diameter 3.2mm")
@@
 	(footprint "Resistor_THT:R_Axial_DIN0309_L9.0mm_D3.2mm_P12.70mm_Horizontal"
 		(layer "F.Cu")
-		(at 138.91 94.14)
+		(at 196.25 126.25 180)
 		(descr "Resistor, Axial_DIN0309 series, Axial, Horizontal, pin pitch=12.7mm, 0.5W = 1/2W, length*diameter=9*3.2mm^2, http://cdn-reichelt.de/documents/datenblatt/B400/1_4W%23YAG.pdf")
 		(tags "Resistor Axial_DIN0309 series Axial Horizontal pin pitch 12.7mm 0.5W = 1/2W length 9mm diameter 3.2mm")
@@
 		(attr through_hole)
 		(fp_line
-			(start 1.04 0)
-			(end 1.73 0)
+			(start 11.66 0)
+			(end 10.97 0)
 			(stroke
 				(width 0.12)
@@
 		)
 		(fp_line
-			(start 11.66 0)
-			(end 10.97 0)
+			(start 1.04 0)
+			(end 1.73 0)
 			(stroke
 				(width 0.12)
@@
 		)
 		(fp_line
-			(start 0 0)
-			(end 1.85 0)
+			(start 12.7 0)
+			(end 10.85 0)
 			(stroke
 				(width 0.1)
@@
 		)
 		(fp_line
-			(start 12.7 0)
-			(end 10.85 0)
+			(start 0 0)
+			(end 1.85 0)
 			(stroke
 				(width 0.1)
@@
 		)
 		(pad "1" thru_hole circle
-			(at 0 0)
+			(at 0 0 180)
 			(size 1.6 1.6)
 			(drill 0.8)
@@
 		)
 		(pad "2" thru_hole circle
-			(at 12.7 0)
+			(at 12.7 0 180)
 			(size 1.6 1.6)
 			(drill 0.8)
@@
 	(footprint "Connector_PinSocket_2.54mm:PinSocket_1x03_P2.54mm_Vertical"
 		(layer "F.Cu")
-		(at 144.26 98.84)
+		(at 191.25 74.67)
 		(descr "Through hole straight socket strip, 1x03, 2.54mm pitch, single row (from Kicad 4.0.7), script generated")
 		(tags "Through hole socket strip THT 1x03 2.54mm single row")
@@
 		)
 	)
+	(segment
+		(start 160.5 97.5)
+		(end 154 97.5)
+		(width 1.2)
+		(layer "F.Cu")
+		(net 6)
+	)
+	(segment
+		(start 178 97.5)
+		(end 171.5 97.5)
+		(width 1.2)
+		(layer "F.Cu")
+		(net 9)
+	)
+	(segment
+		(start 183.55 126.25)
+		(end 178 126.25)
+		(width 1.2)
+		(layer "F.Cu")
+		(net 24)
+	)
+	(segment
+		(start 160.5 102)
+		(end 154 102)
+		(width 1.2)
+		(layer "F.Cu")
+		(net 24)
+	)
+	(segment
+		(start 167.2869 129.1631)
+		(end 170.2 126.25)
+		(width 1.2)
+		(layer "F.Cu")
+		(net 24)
+	)
+	(segment
+		(start 171.5 102)
+		(end 166 102)
+		(width 1.2)
+		(layer "F.Cu")
+		(net 24)
+	)
+	(segment
+		(start 178 126.25)
+		(end 170.2 126.25)
+		(width 1.2)
+		(layer "F.Cu")
+		(net 24)
+	)
+	(segment
+		(start 145 126.75)
+		(end 147.4131 129.1631)
+		(width 1.2)
+		(layer "F.Cu")
+		(net 24)
+	)
+	(segment
+		(start 178 102)
+		(end 171.5 102)
+		(width 1.2)
+		(layer "F.Cu")
+		(net 24)
+	)
+	(segment
+		(start 166 102)
+		(end 160.5 102)
+		(width 1.2)
+		(layer "F.Cu")
+		(net 24)
+	)
+	(segment
+		(start 147.4131 129.1631)
+		(end 167.2869 129.1631)
+		(width 1.2)
+		(layer "F.Cu")
+		(net 24)
+	)
+	(segment
+		(start 178 126.25)
+		(end 178 102)
+		(width 1.2)
+		(layer "F.Cu")
+		(net 24)
+	)
 	(embedded_fonts no)
